File: kicad/pcb/key_matrix.kicad_sch (KiCad schematic)
At the start: 73 parts, among them SW1 SW_Push, SW10 SW_Push, SW11 SW_Push, SW12 SW_Push, SW13 SW_Push, SW14 SW_Push, SW15 SW_Push, SW16 SW_Push, SW17 SW_Push, SW18 SW_Push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

Commit message: More BOM tweaks.
Parts:
- D1, D10, D11, D12, D13, D14, D15, D16, D17, D18, D19, D2, D20, D21, D22, D23, D24, D25, D26, D27, D28, D29, D3, D30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: LCSC (none) -> C908248; MPN (none) -> 1N4148W
- U7, U8, U9: LCSC (none) -> C7666; MPN (none) -> SN74LVC1G08DBVR
