File: kicad/pcb/power.kicad_sch (KiCad schematic)
At the start: 18 parts, among them J4 Conn_01x02_Socket, J5 Conn_01x02_Socket, Q2 AO3401A, U6 MCP73832-2-OT

Commit message: BOM tweaks, switch to horizontal JST SH.
Parts:
- D37: MPN (none) -> BAT54HT1G
- J4: footprint Connector_JST:JST_SH_BM02B-SRSS-TB_1x02-1MP_P1.00mm_Vertical -> Connector_JST:JST_SH_SM02B-SRSS-TB_1x02-1MP_P1.00mm_Horizontal; MPN (none) -> SH-SM02B (SRSS)-TB
- J5, JP3, JP4: now left out of the parts list
- Q2: MPN (none) -> AO3401A
- U6: MPN (none) -> MCP73832-2-OT
- U?: MPN (none) -> XC6206P332PR-G
Changed lines of the file:
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@@
+      (effects (font (size 1.27 1.27)) hide)
+    )
+    (property "MPN" "BAT54HT1G" (at 56.896 147.574 0)
       (effects (font (size 1.27 1.27)) hide)
     )
@@
   )
   (symbol (lib_id "Connector:Conn_01x02_Socket") (at 123.19 112.522 0) (mirror x) (unit 1)
-    (in_bom yes) (on_board yes) (dnp no)
+    (in_bom no) (on_board yes) (dnp no)
     (property "Reference" "J5" (at 124.968 112.522 0)
       (effects (font (size 1.27 1.27)) (justify left))
@@
     (property "Datasheet" "http://www.aosmd.com/pdfs/datasheet/AO3401A.pdf" (at 65.278 137.16 0)
       (effects (font (size 1.27 1.27)) (justify left) hide)
+    )
+    (property "MPN" "AO3401A" (at 65.278 137.16 0)
+      (effects (font (size 1.27 1.27)) hide)
     )
     (pin "2")
@@
       (effects (font (size 1.27 1.27)) hide)
     )
+    (property "MPN" "XC6206P332PR-G" (at 176.022 52.324 0)
+      (effects (font (size 1.27 1.27)) hide)
+    )
     (pin "1")
     (pin "2")
@@
   )
   (symbol (lib_id "Jumper:Jumper_2_Open") (at 139.954 56.896 0) (unit 1)
-    (in_bom yes) (on_board yes) (dnp no) (fields_autoplaced)
+    (in_bom no) (on_board yes) (dnp no) (fields_autoplaced)
     (property "Reference" "JP4" (at 139.954 50.292 0)
       (effects (font (size 1.27 1.27)))
@@
     )
     (property "Datasheet" "http://ww1.microchip.com/downloads/en/DeviceDoc/20001984g.pdf" (at 54.864 87.376 0)
+      (effects (font (size 1.27 1.27)) hide)
+    )
+    (property "MPN" "MCP73832-2-OT" (at 58.674 86.106 0)
       (effects (font (size 1.27 1.27)) hide)
     )
@@
       (effects (font (size 1.27 1.27)) (justify left))
     )
-    (property "Footprint" "Connector_JST:JST_SH_BM02B-SRSS-TB_1x02-1MP_P1.00mm_Vertical" (at 122.682 101.6 0)
+    (property "Footprint" "Connector_JST:JST_SH_SM02B-SRSS-TB_1x02-1MP_P1.00mm_Horizontal" (at 122.682 101.6 0)
       (effects (font (size 1.27 1.27)) hide)
     )
     (property "Datasheet" "~" (at 122.682 101.6 0)
+      (effects (font (size 1.27 1.27)) hide)
+    )
+    (property "MPN" "SH-SM02B (SRSS)-TB" (at 122.682 101.6 0)
       (effects (font (size 1.27 1.27)) hide)
     )
@@
   )
   (symbol (lib_id "Jumper:Jumper_2_Open") (at 139.954 45.466 0) (unit 1)
-    (in_bom yes) (on_board yes) (dnp no) (fields_autoplaced)
+    (in_bom no) (on_board yes) (dnp no) (fields_autoplaced)
     (property "Reference" "JP3" (at 139.954 38.862 0)
       (effects (font (size 1.27 1.27)))

Commit message: More BOM tweaks.
Parts:
- C10, C11: LCSC (none) -> C1779
- C? (x2): LCSC C52923 -> C24123
- D36: LCSC (none) -> C2943978
- D37: LCSC (none) -> C179609
- Q2: LCSC (none) -> C15127
- R3: LCSC (none) -> C2828866
- R4: LCSC (none) -> C100047
- R5: LCSC (none) -> C96346
- R6: LCSC (none) -> C3016844
- R7: LCSC (none) -> C228716; LCSC Part Number (none) -> C228716
- U6: LCSC (none) -> C38066
Changed lines of the file:
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@@
+      (effects (font (size 1.27 1.27)) hide)
+    )
+    (property "LCSC" "C100047" (at 43.18 92.964 0)
       (effects (font (size 1.27 1.27)) hide)
     )
@@
     )
     (property "MPN" "BAT54HT1G" (at 56.896 147.574 0)
+      (effects (font (size 1.27 1.27)) hide)
+    )
+    (property "LCSC" "C179609" (at 56.896 147.574 0)
       (effects (font (size 1.27 1.27)) hide)
     )
@@
       (effects (font (size 1.27 1.27)) hide)
     )
+    (property "LCSC" "C2828866" (at 67.564 72.644 90)
+      (effects (font (size 1.27 1.27)) hide)
+    )
     (pin "2")
     (pin "1")
@@
       (effects (font (size 1.27 1.27)) hide)
     )
+    (property "LCSC" "C96346" (at 47.498 150.876 0)
+      (effects (font (size 1.27 1.27)) hide)
+    )
     (pin "1")
     (pin "2")
@@
     )
     (property "Datasheet" "~" (at 64.77 150.114 0)
+      (effects (font (size 1.27 1.27)) hide)
+    )
+    (property "LCSC" "C1779" (at 64.77 150.114 0)
       (effects (font (size 1.27 1.27)) hide)
     )
@@
       (effects (font (size 1.27 1.27)) hide)
     )
+    (property "LCSC" "C15127" (at 65.278 137.16 0)
+      (effects (font (size 1.27 1.27)) hide)
+    )
     (pin "2")
     (pin "1")
@@
     )
     (property "Datasheet" "~" (at 72.644 86.106 0)
+      (effects (font (size 1.27 1.27)) hide)
+    )
+    (property "LCSC" "C1779" (at 72.644 86.106 0)
       (effects (font (size 1.27 1.27)) hide)
     )
@@
       (effects (font (size 1.27 1.27)) hide)
     )
+    (property "LCSC" "C228716" (at 214.376 101.6 0)
+      (effects (font (size 1.27 1.27)) hide)
+    )
+    (property "LCSC Part Number" "C228716" (at 214.376 101.6 0)
+      (effects (font (size 1.27 1.27)) hide)
+    )
     (pin "2")
     (pin "1")
@@
       (effects (font (size 1.27 1.27)) hide)
     )
+    (property "LCSC" "C38066" (at 58.674 86.106 0)
+      (effects (font (size 1.27 1.27)) hide)
+    )
     (pin "1")
     (pin "4")
@@
     )
     (property "Datasheet" "~" (at 214.376 88.9 0)
+      (effects (font (size 1.27 1.27)) hide)
+    )
+    (property "LCSC" "C3016844" (at 214.376 88.9 0)
       (effects (font (size 1.27 1.27)) hide)
     )
@@
       (effects (font (size 1.27 1.27)) hide)
     )
-    (property "LCSC" "C52923" (at 163.322 56.134 0)
+    (property "LCSC" "C24123" (at 163.322 56.134 0)
       (effects (font (size 1.27 1.27)) hide)
     )
@@
       (effects (font (size 1.27 1.27)) hide)
     )
-    (property "LCSC" "C52923" (at 186.182 56.134 0)
+    (property "LCSC" "C24123" (at 186.182 56.134 0)
       (effects (font (size 1.27 1.27)) hide)
     )
@@
       (effects (font (size 1.27 1.27)) hide)
     )
+    (property "LCSC" "C2943978" (at 77.216 72.644 0)
+      (effects (font (size 1.27 1.27)) hide)
+    )
