File: kicad/pcb/stm32_hotswap_chiffre.kicad_sch (KiCad schematic)
At the start: 22 parts, among them J1 USB_C_Receptacle_USB2.0, J2 SAM, U2 PRTR5V0U2X, U4 ATSAML21E18B-AUT

Commit message: Rework pins to use proper wake/interrupt pins for all matrix outputs, fix edge cuts.
Connections:
- net col0: now also U4.25 (PA27); no longer U4.1 (PA00)
- net col4: now also U4.12 (PA09); no longer U4.3 (PA02)
- net row0_l: now also U4.3 (PA02); no longer U4.12 (PA09)
- net row0_r: now also U4.1 (PA00); no longer U4.25 (PA27)
Changed lines of the file:
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@@
     (effects (font (size 1.27 1.27)) (justify right bottom))
   )
-  (label "PA27" (at 57.15 143.51 0) (fields_autoplaced)
+  (label "PA0" (at 57.15 143.51 0) (fields_autoplaced)
     (effects (font (size 1.27 1.27)) (justify left bottom))
   )
@@
     (effects (font (size 1.27 1.27)) (justify right bottom))
   )
-  (label "PA9" (at 57.15 135.89 0) (fields_autoplaced)
+  (label "PA2" (at 57.15 135.89 0) (fields_autoplaced)
     (effects (font (size 1.27 1.27)) (justify left bottom))
   )
@@
     (effects (font (size 1.27 1.27)) (justify right bottom))
   )
-  (label "PA0" (at 41.402 135.89 0) (fields_autoplaced)
+  (label "PA27" (at 41.402 135.89 0) (fields_autoplaced)
     (effects (font (size 1.27 1.27)) (justify left bottom))
   )
@@
     (effects (font (size 1.27 1.27)) (justify left bottom))
   )
-  (label "PA2" (at 41.402 146.05 0) (fields_autoplaced)
+  (label "PA9" (at 41.402 146.05 0) (fields_autoplaced)
     (effects (font (size 1.27 1.27)) (justify left bottom))
   )

Commit message: BOM tweaks, switch to horizontal JST SH.
Parts:
- J2, JP2: now left out of the parts list
Changed lines of the file:
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@@
   )
   (symbol (lib_id "Jumper:Jumper_2_Open") (at 46.482 44.704 0) (unit 1)
-    (in_bom yes) (on_board yes) (dnp no) (fields_autoplaced)
+    (in_bom no) (on_board yes) (dnp no) (fields_autoplaced)
     (property "Reference" "JP2" (at 46.482 38.1 0)
       (effects (font (size 1.27 1.27)))
@@
   )
   (symbol (lib_id "PCM_marbastlib-various:TC2030_SWD") (at 128.016 104.648 0) (unit 1)
-    (in_bom yes) (on_board yes) (dnp no) (fields_autoplaced)
+    (in_bom no) (on_board yes) (dnp no) (fields_autoplaced)
     (property "Reference" "J2" (at 135.382 102.108 0)
       (effects (font (size 1.27 1.27)) (justify left))

Commit message: More BOM tweaks.
Parts:
- C5: LCSC (none) -> C24123
- C? (x3): LCSC C307331 -> C38141
- C?: LCSC (none) -> C17024
- C?: LCSC C307331 -> C17024
- D38: LCSC (none) -> C84259
- F1: value ASMD1206-150 -> 500mA; LCSC C135341 -> C883119; MPN (none) -> BSMD1206-025-16V
- J1: MPN (none) -> TYPE-C-31-M-12
- L1: LCSC C33600 -> C3033915; MPN (none) -> MLB3216-600P4A(f); Manufacturer Part No MLB3216-600P4A(f) -> (none)
- L2: LCSC (none) -> C139245; LCSC Part Number C2932309 -> (none)
- R10: LCSC (none) -> C2907256
- R11: LCSC (none) -> C95781
- R8: LCSC (none) -> C228716
- R9: LCSC (none) -> C2828721
- R? (x2): LCSC (none) -> C118848
- U2: MPN (none) -> PRTR5V0U2X
- U4: LCSC (none) -> C2053723; MPN (none) -> ATSAML21E18B-AUT
Changed lines of the file:
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@@
+      (effects (font (size 1.27 1.27)) hide)
+    )
+    (property "LCSC" "C2907256" (at 96.012 108.712 0)
       (effects (font (size 1.27 1.27)) hide)
     )
@@
       (effects (font (size 1.27 1.27)) hide)
     )
-    (property "Manufacturer Part No" "MLB3216-600P4A(f)" (at 201.93 60.96 0)
-      (effects (font (size 1.27 1.27)) hide)
-    )
-    (property "LCSC" "C33600" (at 201.93 60.96 0)
+    (property "Manufacturer Part No" "" (at 201.93 60.96 0)
+      (effects (font (size 1.27 1.27)) hide)
+    )
+    (property "LCSC" "C3033915" (at 201.93 60.96 0)
       (effects (font (size 1.27 1.27)) hide)
     )
     (property "Package" "L1206" (at 201.93 60.96 0)
+      (effects (font (size 1.27 1.27)) hide)
+    )
+    (property "MPN" "MLB3216-600P4A(f)" (at 201.93 60.96 0)
       (effects (font (size 1.27 1.27)) hide)
     )
@@
     )
     (property "JlcPosOffset" "0,1.5" (at 167.64 48.26 0)
+      (effects (font (size 1.27 1.27)) hide)
+    )
+    (property "MPN" "TYPE-C-31-M-12" (at 167.64 48.26 0)
       (effects (font (size 1.27 1.27)) hide)
     )
@@
       (effects (font (size 1.27 1.27)) hide)
     )
+    (property "MPN" "PRTR5V0U2X" (at 183.642 113.03 0)
+      (effects (font (size 1.27 1.27)) hide)
+    )
     (pin "1")
     (pin "2")
@@
     )
     (property "Datasheet" "http://ww1.microchip.com/downloads/en/DeviceDoc/60001477A.pdf" (at 46.736 87.376 0)
+      (effects (font (size 1.27 1.27)) hide)
+    )
+    (property "MPN" "ATSAML21E18B-AUT" (at 46.736 87.376 0)
+      (effects (font (size 1.27 1.27)) hide)
+    )
+    (property "LCSC" "C2053723" (at 46.736 87.376 0)
       (effects (font (size 1.27 1.27)) hide)
     )
@@
       (effects (font (size 1.27 1.27)) hide)
     )
+    (property "LCSC" "C118848" (at 186.69 40.64 0)
+      (effects (font (size 1.27 1.27)) hide)
+    )
     (pin "1")
     (pin "2")
@@
       (effects (font (size 1.27 1.27)) hide)
     )
-    (property "LCSC Part Number" "C2932309" (at 47.244 53.848 90)
+    (property "LCSC Part Number" "" (at 47.244 53.848 90)
+      (effects (font (size 1.27 1.27)) hide)
+    )
+    (property "LCSC" "C139245" (at 47.244 53.848 0)
       (effects (font (size 1.27 1.27)) hide)
     )
@@
       (effects (font (size 1.27 1.27)) hide)
     )
-    (property "LCSC" "C307331" (at 73.66 37.592 0)
+    (property "LCSC" "C38141" (at 73.66 37.592 0)
       (effects (font (size 1.27 1.27)) hide)
     )
@@
       (effects (font (size 1.27 1.27)) hide)
     )
-    (property "LCSC" "" (at 130.81 37.592 0)
+    (property "LCSC" "C17024" (at 130.81 37.592 0)
       (effects (font (size 1.27 1.27)) hide)
     )
@@
       (effects (font (size 1.27 1.27)) hide)
     )
-    (property "LCSC" "C307331" (at 85.09 37.592 0)
+    (property "LCSC" "C38141" (at 85.09 37.592 0)
       (effects (font (size 1.27 1.27)) hide)
     )
@@
       (effects (font (size 1.27 1.27)))
     )
-    (property "Value" "ASMD1206-150" (at 172.212 94.742 90)
+    (property "Value" "500mA" (at 172.212 94.742 90)
       (effects (font (size 1.27 1.27)))
     )
@@
       (effects (font (size 1.27 1.27)) hide)
     )
-    (property "LCSC" "C135341" (at 172.212 97.282 90)
+    (property "LCSC" "C883119" (at 172.212 97.282 90)
+      (effects (font (size 1.27 1.27)) hide)
+    )
+    (property "MPN" "BSMD1206-025-16V" (at 172.212 97.282 0)
       (effects (font (size 1.27 1.27)) hide)
     )
@@
       (effects (font (size 1.27 1.27)) hide)
     )
+    (property "LCSC" "C84259" (at 96.012 103.632 0)
+      (effects (font (size 1.27 1.27)) hide)
+    )
     (pin "2")
     (pin "1")
@@
     )
     (property "Datasheet" "~" (at 186.69 38.1 0)
+      (effects (font (size 1.27 1.27)) hide)
+    )
+    (property "LCSC" "C118848" (at 186.69 38.1 0)
       (effects (font (size 1.27 1.27)) hide)
     )
@@
       (effects (font (size 1.27 1.27)) hide)
     )
-    (property "LCSC" "C307331" (at 203.962 101.092 0)
+    (property "LCSC" "C38141" (at 203.962 101.092 0)
       (effects (font (size 1.27 1.27)) hide)
     )
@@
       (effects (font (size 1.27 1.27)) hide)
     )
+    (property "LCSC" "C2828721" (at 98.298 82.042 0)
+      (effects (font (size 1.27 1.27)) hide)
+    )
     (pin "2")
     (pin "1")
@@
       (effects (font (size 1.27 1.27)) hide)
     )
-    (property "LCSC" "C307331" (at 119.38 37.592 0)
+    (property "LCSC" "C17024" (at 119.38 37.592 0)
       (effects (font (size 1.27 1.27)) hide)
     )
@@
       (effects (font (size 1.27 1.27)) hide)
     )
+    (property "LCSC" "C24123" (at 40.894 58.166 0)
+      (effects (font (size 1.27 1.27)) hide)
+    )
     (pin "2")
     (pin "1")
@@
       (effects (font (size 1.27 1.27)) hide)
     )
+    (property "LCSC" "C95781" (at 112.014 94.488 0)
+      (effects (font (size 1.27 1.27)) hide)
+    )
     (pin "2")
     (pin "1")
@@
       (effects (font (size 1.27 1.27)) hide)
     )
+    (property "LCSC" "C228716" (at 98.298 71.628 0)
+      (effects (font (size 1.27 1.27)) hide)
+    )
