File: kicad/pcb/wireless.kicad_sch (KiCad schematic)
At the start: 6 parts, among them J3 nRF52, U5 BC805M, Y2 32.768 kHz

Commit message: BOM tweaks, switch to horizontal JST SH.
Parts:
- J3: now left out of the parts list
Changed lines of the file:
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@@
   )
   (symbol (lib_id "PCM_marbastlib-various:TC2030_SWD") (at 214.63 56.642 0) (unit 1)
-    (in_bom yes) (on_board yes) (dnp no) (fields_autoplaced)
+    (in_bom no) (on_board yes) (dnp no) (fields_autoplaced)
     (property "Reference" "J3" (at 222.25 54.102 0)
       (effects (font (size 1.27 1.27)) (justify left))

Commit message: More BOM tweaks.
Parts:
- C12, C13: LCSC (none) -> C1792
- C6: LCSC (none) -> C17024
- U5: LCSC (none) -> C6751361; MPN (none) -> BC805M
- Y2: value 32.768 kHz -> 32.768 kHz 12.5pF ±20ppm; LCSC (none) -> C97603
Changed lines of the file:
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@@
       (effects (font (size 1.524 1.524)) hide)
+    )
+    (property "MPN" "BC805M" (at 99.568 42.164 0)
+      (effects (font (size 1.27 1.27)) hide)
+    )
+    (property "LCSC" "C6751361" (at 99.568 42.164 0)
+      (effects (font (size 1.27 1.27)) hide)
     )
     (pin "3")
@@
       (effects (font (size 1.27 1.27)) (justify right))
     )
-    (property "Value" "32.768 kHz" (at 153.67 35.56 90)
+    (property "Value" "32.768 kHz 12.5pF ±20ppm" (at 153.67 35.56 90)
       (effects (font (size 1.27 1.27)) (justify right))
     )
@@
       (effects (font (size 1.27 1.27)) hide)
     )
+    (property "LCSC" "C97603" (at 151.13 34.29 0)
+      (effects (font (size 1.27 1.27)) hide)
+    )
     (pin "1")
     (pin "2")
@@
       (effects (font (size 1.27 1.27)) hide)
     )
+    (property "LCSC" "C17024" (at 131.572 48.514 0)
+      (effects (font (size 1.27 1.27)) hide)
+    )
     (pin "2")
     (pin "1")
@@
       (effects (font (size 1.27 1.27)) hide)
     )
+    (property "LCSC" "C1792" (at 161.036 39.37 0)
+      (effects (font (size 1.27 1.27)) hide)
+    )
     (pin "1")
     (pin "2")
@@
       (effects (font (size 1.27 1.27)) hide)
     )
+    (property "LCSC" "C1792" (at 160.782 29.21 0)
+      (effects (font (size 1.27 1.27)) hide)
+    )
